File: rev2/rev2.kicad_pcb (KiCad board)
At the start: 2 copper layers, 133.3 x 91.2 mm, 74 parts, among them J101 Bluefruit LE, J102 Display, J103 JST-PH, SW101 Y, SW102 U, SW103 I, SW104 O, SW105 P, SW106 BSPC, SW107 H, SW108 J, SW109 K, SW110 L, SW111 ;, SW112 ENT, SW113 N, SW114 M, SW115 ,, SW116 ., SW117 /, SW118 RSHIFT, SW119 SPC, SW120 M1, SW121 M2, SW122 SUPER, U101 ATmega32U4, Y101 16 MHz

Commit message: revision 1 and 2 added
Parts:
- removed H105: MountingHole_Pad, MountingHole:MountingHole_2.2mm_M2_Pad_TopBottom
- removed J102: Display, Connector_PinHeader_2.54mm:PinHeader_1x04_P2.54mm_Vertical
- removed JP101, JP102, JP103: Voltage Sense, Jumper:SolderJumper-2_P1.3mm_Open_Pad1.0x1.5mm
- added D101: D, Diode_SMD:D_0603_1608Metric, B.Cu at (54.1, 37.1)
- added D102: D, Diode_SMD:D_0603_1608Metric, B.Cu at (73.1, 34.6)
- added D103: D, Diode_SMD:D_0603_1608Metric, B.Cu at (92.2, 29.5)
- added D104: D, Diode_SMD:D_0603_1608Metric, B.Cu at (111.2, 34.6)
- added D105: D, Diode_SMD:D_0603_1608Metric, B.Cu at (130.3, 44.6)
- added D106: D, Diode_SMD:D_0603_1608Metric, B.Cu at (149.3, 44.7)
- added D107: D, Diode_SMD:D_0603_1608Metric, B.Cu at (35.0, 39.5)
- added D114: D, Diode_SMD:D_0603_1608Metric, B.Cu at (35.1, 58.7)
- added D121: D, Diode_SMD:D_0603_1608Metric, B.Cu at (35.0, 77.7)
- added D128: D, Diode_SMD:D_0603_1608Metric, B.Cu at (35.0, 96.8)
- added SW101: 6, CherryMX_PCB:CherryMX_1.00u_PCB, F.Cu at (60.3, 42.5)
- added SW102: 7, CherryMX_PCB:CherryMX_1.00u_PCB, F.Cu at (79.4, 40.0)
- added SW103: 8, CherryMX_PCB:CherryMX_1.00u_PCB, F.Cu at (98.4, 34.9)
- added SW104: 9, CherryMX_PCB:CherryMX_1.00u_PCB, F.Cu at (117.5, 40.0)
- added SW105: 0, CherryMX_PCB:CherryMX_1.00u_PCB, F.Cu at (136.5, 50.2)
- added SW106: -, CherryMX_PCB:CherryMX_1.00u_PCB, F.Cu at (155.6, 50.2)
- added SW107: C1, CherryMX_PCB:CherryMX_1.00u_PCB, F.Cu at (41.3, 45.1)
- added SW114: C2, CherryMX_PCB:CherryMX_1.00u_PCB, F.Cu at (41.3, 64.1)
- added SW121: C3, CherryMX_PCB:CherryMX_1.00u_PCB, F.Cu at (41.3, 83.2)
- added SW128: C4, CherryMX_PCB:CherryMX_1.00u_PCB, F.Cu at (41.3, 102.2)
- C101, C102, C103, C104, C105, C106, C107, C108, R101: moved to B.Cu
- J101: footprint Connector_PinHeader_2.54mm:PinHeader_1x09_P2.54mm_Vertical -> Connector_JST:JST_SH_SM08B-SRSS-TB_1x08-1MP_P1.00mm_Horizontal
- J103: footprint Connector_JST:JST_PH_S4B-PH-SM4-TB_1x04-1MP_P2.00mm_Horizontal -> Connector_JST:JST_SH_SM04B-SRSS-TB_1x04-1MP_P1.00mm_Horizontal
- R104: renamed from R102; moved to B.Cu
- R107: renamed from R103; moved to B.Cu
- R108: renamed from R106; moved to B.Cu
- moved D108 136.3 mm to (54.1, 56.1), turned to -90 degrees
- moved D129 135.3 mm to (54.4, 127.7), turned to 105 degrees
- moved D115 131.5 mm to (54.1, 75.2), turned to -90 degrees
- moved D122 129.4 mm to (54.1, 94.3), turned to -90 degrees
- moved R101 120.2 mm to (78.0, 106.7), turned to -90 degrees
- moved D109 118.2 mm to (73.2, 53.6), turned to -90 degrees
- moved D130 115.4 mm to (73.5, 124.0), turned to 100 degrees
- moved D116 112.4 mm to (73.2, 72.7), turned to -90 degrees
- moved D123 109.8 mm to (73.2, 91.7), turned to -90 degrees
- moved C106 109.6 mm to (92.9, 120.0), turned to -45 degrees
- moved R104 107.7 mm to (86.6, 98.0), turned to 90 degrees
- moved D131 107.6 mm to (80.4, 123.1), turned to 95 degrees
- moved C107 104.0 mm to (97.4, 119.3), turned to -135 degrees
- moved C103 103.6 mm to (86.2, 106.9), turned to -90 degrees
- moved R107 103.4 mm to (86.0, 85.9), turned to -90 degrees
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- renumbered D101 to D108, D102 to D109, D103 to D110, D104 to D111, D105 to D112, D106 to D113, D107 to D115, D108 to D116, D109 to D117, D110 to D118, D111 to D119, D112 to D120, D113 to D122, D114 to D123, D115 to D124, D116 to D125, D117 to D126, D118 to D127, D119 to D129, D120 to D130, D121 to D131, D122 to D132, D123 to D133, D124 to D134, R104 to R105, R105 to R106, SW101 to SW108, SW102 to SW109, SW103 to SW110, SW104 to SW111, SW105 to SW112, SW106 to SW113, SW107 to SW115, SW108 to SW116, SW109 to SW117, SW110 to SW118, SW111 to SW119, SW112 to SW120, SW113 to SW122, SW114 to SW123, SW115 to SW124, SW116 to SW125, SW117 to SW126, SW118 to SW127, SW119 to SW129, SW120 to SW130, SW121 to SW131, SW122 to SW132
Connections:
- D108 pad 1: row_0 -> row_1
- D109 pad 1: row_0 -> row_1
- D110 pad 1: row_0 -> row_1
- D111 pad 1: row_0 -> row_1
- D112 pad 1: row_0 -> row_1
- D113 pad 1: row_0 -> row_1
- D115 pad 1: row_1 -> row_2
- D116 pad 1: row_1 -> row_2
- D117 pad 1: row_1 -> row_2
- D118 pad 1: row_1 -> row_2
- D119 pad 1: row_1 -> row_2
- D120 pad 1: row_1 -> row_2
- D122 pad 1: row_2 -> row_3
- D123 pad 1: row_2 -> row_3
- D124 pad 1: row_2 -> row_3
- D125 pad 1: row_2 -> row_3
- D126 pad 1: row_2 -> row_3
- D127 pad 1: row_2 -> row_3
- D129 pad 1: row_3 -> row_4
- D130 pad 1: row_3 -> row_4
- D131 pad 1: row_3 -> row_4
- D132 pad 1: row_3 -> row_4
- D133 pad 2: Net-(D123-A) (its old number) -> Net-(D133-A)
- D134 pad 2: Net-(D124-A) (its old number) -> Net-(D134-A)
- J101 pad 4: unconnected-(J101-Pin_4-Pad4) -> BLE_IRQ
- J101 pad 5: BLE_IRQ -> BLE_CS
- J101 pad 6: BLE_CS -> MOSI
- J101 pad 7: MOSI -> MISO
- J101 pad 8: MISO -> SCK
- R107 pad 2: Net-(JP101-A) -> Net-(D133-A)
- R108 pad 2: Net-(JP102-A) -> Net-(D134-A)
- SW129 pad 2: col_2 -> col_0
- SW130 pad 2: col_3 -> col_1
- SW131 pad 2: col_4 -> col_3
- SW132 pad 2: col_5 -> col_4
- U101 pad 1: BLE_IRQ -> BLE_RST
- U101 pad 12: col_5 -> row_4
- U101 pad 18: SCL -> unconnected-(U101-PD0-Pad18)
- U101 pad 19: SDA -> col_4
- U101 pad 20: unconnected-(U101-PD2-Pad20) -> col_5
- U101 pad 21: col_0 -> col_3
- U101 pad 22: unconnected-(U101-PD5-Pad22) -> col_6
- U101 pad 25: BLE_RST -> col_2
- U101 pad 27: col_2 -> col_0
- U101 pad 28: BLE_CS -> unconnected-(U101-PB4-Pad28)
- U101 pad 29: col_3 -> row_0
- U101 pad 30: col_4 -> row_1
- U101 pad 31: unconnected-(U101-PC6-Pad31) -> row_2
- U101 pad 32: unconnected-(U101-PC7-Pad32) -> row_3
- U101 pad 37: row_3 -> unconnected-(U101-PF6-Pad37)
- U101 pad 38: row_2 -> unconnected-(U101-PF5-Pad38)
- U101 pad 39: row_1 -> unconnected-(U101-PF4-Pad39)
- U101 pad 40: row_0 -> BLE_IRQ
- U101 pad 41: ADC_VBAT -> unconnected-(U101-PF0-Pad41)
- U101 pad 8: unconnected-(U101-PB0-Pad8) -> BLE_CS
Routing:
- net VCC: track 0.00 -> 244.0 mm, vias 0 -> 2
- net row_0: track 0.00 -> 241.0 mm, vias 0 -> 4
- net row_1: track 0.00 -> 203.1 mm, vias 0 -> 4
- net row_2: track 0.00 -> 188.2 mm, vias 0 -> 6
- net row_3: track 0.00 -> 163.4 mm, vias 0 -> 4
- net col_5: track 0.00 -> 162.6 mm, vias 0 -> 1
- net col_4: track 0.00 -> 141.2 mm, vias 0 -> 1
- net col_0: track 0.00 -> 138.4 mm, vias 0 -> 1
- net col_3: track 0.00 -> 113.9 mm
- net col_6: track 0.00 -> 109.0 mm
- net col_1: track 0.00 -> 102.1 mm, vias 0 -> 1
- net col_2: track 0.00 -> 89.9 mm, vias 0 -> 1
- net BLE_CS: track 0.00 -> 75.8 mm, vias 0 -> 2
- net MISO: track 0.00 -> 74.2 mm
- net SCK: track 0.00 -> 73.8 mm
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- added copper zone on B.Cu, net GND
- added copper zone on F.Cu, net GND
Other:
- board size 133.3 x 91.2 mm -> 133.3 x 110.2 mm
- board text added: "BLUEFRUIT"
- board text added: "KH"
- board text added: "MCU"
- board text added: "R"
- board text added: "RESET"
- board text added: "USB"
- board text added: "VCC"
- board text added: "rev 2.0"
- board text removed: "OLED"

Commit message: updated some stuff
Parts:
- D101, D102, D103, D104, D105, D106, D107, D108, D109, D110, D111, D112, D113, D114, D115, D116, D117, D118, D119, D120, D121, D122, D123, D124, D125, D126, D127, D128, D129, D130, D131, D132: footprint Diode_SMD:D_0603_1608Metric -> Diode_SMD:D_SOD-123
- moved D132 0.97 mm to (103.9, 110.6)
- moved D123 0.92 mm to (73.4, 90.8)
- moved D107 0.42 mm to (34.9, 39.1)
Routing:
- net row_1: track 203.1 -> 200.0 mm
- net row_4: track 68.4 -> 70.6 mm
- net row_3: track 163.4 -> 165.3 mm
- net row_2: track 188.2 -> 186.6 mm
- net row_0: track 241.0 -> 239.7 mm
- net Net-(D113-A): track 4.61 -> 5.22 mm
