File: usb-board/usb-board.kicad_sch (KiCad schematic)
At the start: 19 parts, among them J101 Conn_01x04_MountingPin, J102 USB_C_2.0, J103 Battery_Conn, SW101 PCM13SMTR, U101 MCP73831-2-OT

Commit message: revision 1 and 2 added
Parts:
- removed H102: MountingHole_Pad, MountingHole:MountingHole_2.2mm_M2_Pad, symbol Mechanical:MountingHole_Pad
- J101: footprint Connector_JST:JST_PH_S4B-PH-SM4-TB_1x04-1MP_P2.00mm_Horizontal -> Connector_JST:JST_SH_SM04B-SRSS-TB_1x04-1MP_P1.00mm_Horizontal
- R105: value 5k -> 5.1k
- renumbered H104 to H102
Connections:
- net VCC: now also SW101.1; no longer SW101.4
- net at C104.1, U101.3 (V_{BAT}): now also SW101.4; no longer SW101.2
Other:
- moved on the sheet: C104, H102
