File: rev2-left/rev2-left.kicad_pcb (KiCad board)
At the start: 2 copper layers, 133.4 x 110.2 mm, 89 parts, among them J101 Bluefruit LE, J102 JST-PH, SW101 ESC, SW102 1, SW103 2, SW104 3, SW105 4, SW106 5, SW107 C1, SW108 TAB, SW109 Q, SW110 W, SW111 E, SW112 R, SW113 T, SW114 C2, SW115 LSHIFT, SW116 A, SW117 S, SW118 D, SW119 F, SW120 G, SW121 C3, SW122 LCTRL, SW123 Z, SW124 X, SW125 C, SW126 V, SW127 B, SW128 C4, SW129 SUPER, SW130 M1, SW131 M2, SW132 SPACE, U101 ATmega32U4, Y101 16 MHz

Commit message: updated some stuff
Parts:
- D101, D102, D103, D104, D105, D106, D107, D108, D109, D110, D111, D112, D113, D114, D115, D116, D117, D118, D119, D120, D121, D122, D123, D124, D125, D126, D127, D128, D129, D130, D131, D132: footprint Diode_SMD:D_0603_1608Metric -> Diode_SMD:D_SOD-123
- moved D116 3.28 mm to (64.6, 91.7), turned to -90 degrees
- moved H104 0.77 mm to (63.5, 97.8)
Routing:
- net Net-(D116-A): track 4.68 -> 10.1 mm
- net Net-(D129-A): track 15.0 -> 13.3 mm
- net Net-(D130-A): track 14.2 -> 13.3 mm
- net row_2: track 194.5 -> 193.8 mm
- net row_4: track 68.7 -> 68.1 mm
